File: lightningbug.sch (EAGLE design)
At the start: 24 parts, among them U1 LV321SOT23-5, U2 LV321SOT23-5, U3 LV321SOT23-5

Commit message: schematic in process
Parts:
- removed I?C2: 10uF, LITTLEBITS:CAPCAP-0603
- removed I?R3, I?R4: 3K3, LITTLEBITS:RESISTOR0603
- added POTD, POTF: 10kPOT, LITTLEBITS140915:POT-TRIM-SMD-BOURNS-3303
- added SWITCHD, SWITCHF: AYZ0202, LITTLEBITS140915:AYZ0202
- added U$3: ATTINY85, LITTLEBITS140915:ATTINY85
- added W2R3: 10k, LITTLEBITS:CAPCAP-0603
Connections:
- removed net N$1: U1.+IN
- removed net N$4: U2.+IN
- removed net N$5: U3.+IN
- removed net VREF: I?C2.1, I?R3.1, I?R4.2
- new net N$6: U$3.PB5(NRES), W2R3.2
- new net OUT1: U$3.PB4(ADC2), U1.+IN
- new net OUT2: U$3.PB0(MOSI), U2.+IN
- new net OUT3: U$3.PB1(MISO), U3.+IN
- net GND: now also POTD.1, POTF.1, U$3.GND; no longer I?C2.2, I?R4.1
- net N$2: now also U$3.VCC, W2R3.1
- net VCC: now also POTD.3, POTF.3; no longer I?R3.2
Other:
- note removed: "IF YOU NEED A VREF:"
- note removed: "TYPICAL POWER SECTION"
Changed lines of the file:
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@@
 <part name="W2TVS1" library="LITTLEBITS" deviceset="DIODE-TVS" device="SOD-923" value="ESD9B5.0ST5G"/>
 <part name="GND9" library="SparkFun" deviceset="GND" device=""/>
-<part name="P+8" library="SparkFun" deviceset="VCC" device=""/>
-<part name="I?R3" library="LITTLEBITS" deviceset="RESISTOR" device="0603" value="3K3">
-<attribute name="COMPOSITION" value=""/>
-<attribute name="LB_PN" value=""/>
-<attribute name="POWER" value=""/>
-<attribute name="TOLERANCE" value=""/>
-</part>
-<part name="I?R4" library="LITTLEBITS" deviceset="RESISTOR" device="0603" value="3K3">
-<attribute name="COMPOSITION" value=""/>
-<attribute name="LB_PN" value=""/>
-<attribute name="POWER" value=""/>
-<attribute name="TOLERANCE" value=""/>
-</part>
 <part name="I?C1" library="LITTLEBITS" deviceset="CAP" device="CAP-0603" value="0.1uF"/>
 <part name="U3" library="LITTLEBITS" deviceset="LV321" device="SOT23-5"/>
@@
 <part name="P+11" library="SparkFun" deviceset="VCC" device=""/>
 <part name="GND15" library="SparkFun" deviceset="GND" device=""/>
-<part name="I?C2" library="LITTLEBITS" deviceset="CAP" device="CAP-0603" value="10uF"/>
 <part name="GND6" library="SparkFun" deviceset="GND" device=""/>
 <part name="GND7" library="SparkFun" deviceset="GND" device=""/>
@@
 <part name="U$1" library="LITTLEBITS" deviceset="OSHWCREDIT" device=""/>
 <part name="FRAME1" library="LITTLEBITS" deviceset="FRAME-LETTER" device=""/>
+<part name="U$3" library="LITTLEBITS140915" deviceset="ATTINY85" device=""/>
+<part name="SWITCHD" library="LITTLEBITS140915" deviceset="AYZ0202" device=""/>
+<part name="SWITCHF" library="LITTLEBITS140915" deviceset="AYZ0202" device=""/>
+<part name="POTF" library="LITTLEBITS140915" deviceset="POT-TRIM-SMD-BOURNS-3303" device="" value="10kPOT"/>
+<part name="POTD" library="LITTLEBITS140915" deviceset="POT-TRIM-SMD-BOURNS-3303" device="" value="10kPOT"/>
+<part name="W2R3" library="LITTLEBITS" deviceset="CAP" device="CAP-0603" value="10k"/>
+<part name="GND18" library="SparkFun" deviceset="GND" device=""/>
+<part name="GND19" library="SparkFun" deviceset="GND" device=""/>
+<part name="P+8" library="SparkFun" deviceset="VCC" device=""/>
+<part name="P+14" library="SparkFun" deviceset="VCC" device=""/>
 </parts>
 <sheets>
@@
 <text x="7.62" y="30.48" size="1.778" layer="91">TYPICAL CONNECTION IS TO VCC OR GND.</text>
 <text x="7.62" y="43.18" size="1.778" layer="91">TYPICAL INPUT SECTION:</text>
-<text x="109.22" y="182.88" size="1.778" layer="91">TYPICAL POWER SECTION</text>
-<text x="109.22" y="180.34" size="1.778" layer="91">IF YOU NEED A VREF:</text>
 <text x="187.96" y="43.18" size="1.778" layer="91">TVS PROVIDES ESD PROTECTION.</text>
 <text x="12.7" y="60.96" size="1.778" layer="91">BYPASS EVERY IC</text>
@@
 <instance part="W2R2" gate="G$1" x="48.26" y="99.06"/>
 <instance part="W2TVS1" gate="G$1" x="35.56" y="96.52"/>
-<instance part="GND9" gate="1" x="129.54" y="139.7"/>
-<instance part="P+8" gate="1" x="121.92" y="170.18"/>
-<instance part="I?R3" gate="G$1" x="121.92" y="162.56" rot="R90"/>
-<instance part="I?R4" gate="G$1" x="121.92" y="149.86" rot="R90"/>
+<instance part="GND9" gate="1" x="91.44" y="81.28"/>
 <instance part="I?C1" gate="G$1" x="10.16" y="58.42" smashed="yes">
 <attribute name="NAME" x="4.064" y="61.341" size="1.778" layer="95"/>
@@
 <instance part="P+11" gate="1" x="10.16" y="66.04"/>
 <instance part="GND15" gate="1" x="10.16" y="50.8"/>
-<instance part="I?C2" gate="G$1" x="129.54" y="147.32"/>
 <instance part="GND6" gate="1" x="22.86" y="81.28"/>
 <instance part="GND7" gate="1" x="35.56" y="81.28"/>
@@
 <instance part="FRAME1" gate="G$1" x="0" y="0"/>
 <instance part="FRAME1" gate="G$2" x="147.32" y="0"/>
+<instance part="U$3" gate="G$1" x="106.68" y="88.9"/>
+<instance part="SWITCHD" gate="G$1" x="114.3" y="50.8"/>
+<instance part="SWITCHF" gate="G$1" x="119.38" y="121.92"/>
+<instance part="POTF" gate="G$1" x="96.52" y="121.92"/>
+<instance part="POTD" gate="G$1" x="139.7" y="60.96"/>
+<instance part="W2R3" gate="G$1" x="104.14" y="73.66" rot="R90"/>
+<instance part="GND18" gate="1" x="96.52" y="111.76"/>
+<instance part="GND19" gate="1" x="139.7" y="50.8"/>
+<instance part="P+8" gate="1" x="96.52" y="129.54"/>
+<instance part="P+14" gate="1" x="139.7" y="68.58"/>
 </instances>
 <busses>
@@
 <pinref part="W2U1" gate="G$1" pin="-IN"/>
 <pinref part="W2U1" gate="G$1" pin="OUT"/>
-<wire x1="73.66" y1="96.52" x2="96.52" y2="96.52" width="0.1524" layer="91"/>
+<wire x1="73.66" y1="96.52" x2="83.82" y2="96.52" width="0.1524" layer="91"/>
 <junction x="73.66" y="96.52"/>
+<pinref part="U$3" gate="G$1" pin="VCC"/>
+<wire x1="83.82" y1="96.52" x2="91.44" y2="96.52" width="0.1524" layer="91"/>
+<wire x1="83.82" y1="96.52" x2="83.82" y2="73.66" width="0.1524" layer="91"/>
+<pinref part="W2R3" gate="G$1" pin="1"/>
+<wire x1="83.82" y1="73.66" x2="99.06" y2="73.66" width="0.1524" layer="91"/>
+<junction x="83.82" y="96.52"/>
 </segment>
 </net>
@@
 </segment>
 <segment>
-<pinref part="P+8" gate="1" pin="VCC"/>
-<pinref part="I?R3" gate="G$1" pin="2"/>
-<wire x1="121.92" y1="167.64" x2="121.92" y2="170.18" width="0.1524" layer="91"/>
-</segment>
-<segment>
 <pinref part="U3" gate="G$1" pin="V+"/>
 <pinref part="P+10" gate="1" pin="VCC"/>
@@
 <wire x1="152.4" y1="152.4" x2="152.4" y2="149.86" width="0.1524" layer="91"/>
 </segment>
+<segment>
+<pinref part="POTF" gate="G$1" pin="3"/>
+<pinref part="P+8" gate="1" pin="VCC"/>
+</segment>
+<segment>
+<pinref part="POTD" gate="G$1" pin="3"/>
+<pinref part="P+14" gate="1" pin="VCC"/>
+</segment>
 </net>
 <net name="GND" class="0">
@@
 </segment>
 <segment>
-<pinref part="I?R4" gate="G$1" pin="1"/>
-<pinref part="GND9" gate="1" pin="GND"/>
-<wire x1="129.54" y1="142.24" x2="121.92" y2="142.24" width="0.1524" layer="91"/>
-<wire x1="121.92" y1="142.24" x2="121.92" y2="144.78" width="0.1524" layer="91"/>
-<wire x1="129.54" y1="142.24" x2="129.54" y2="144.78" width="0.1524" layer="91"/>
-<junction x="129.54" y="142.24"/>
-<pinref part="I?C2" gate="G$1" pin="2"/>
-</segment>
-<segment>
 <pinref part="U3" gate="G$1" pin="V-"/>
 <pinref part="GND12" gate="1" pin="GND"/>
@@
 <pinref part="GND14" gate="1" pin="GND"/>
 </segment>
-</net>
-<net name="VREF" class="0">
-<segment>
-<pinref part="I?R3" gate="G$1" pin="1"/>
-<pinref part="I?R4" gate="G$1" pin="2"/>
-<wire x1="121.92" y1="154.94" x2="121.92" y2="157.48" width="0.1524" layer="91"/>
-<wire x1="121.92" y1="154.94" x2="129.54" y2="154.94" width="0.1524" layer="91"/>
-<junction x="121.92" y="154.94"/>
-<wire x1="129.54" y1="152.4" x2="129.54" y2="154.94" width="0.1524" layer="91"/>
-<wire x1="129.54" y1="154.94" x2="137.16" y2="154.94" width="0.1524" layer="91"/>
-<label x="137.16" y="154.94" size="1.778" layer="95" xref="yes"/>
-<junction x="129.54" y="154.94"/>
-<pinref part="I?C2" gate="G$1" pin="1"/>
+<segment>
+<pinref part="U$3" gate="G$1" pin="GND"/>
+<pinref part="GND9" gate="1" pin="GND"/>
+</segment>
+<segment>
+<pinref part="POTF" gate="G$1" pin="1"/>
+<pinref part="GND18" gate="1" pin="GND"/>
+</segment>
+<segment>
+<pinref part="POTD" gate="G$1" pin="1"/>
+<pinref part="GND19" gate="1" pin="GND"/>
 </segment>
 </net>
@@
 </segment>
 </net>
-<net name="N$5" class="0">
+<net name="OUT3" class="0">
 <segment>
 <pinref part="U3" gate="G$1" pin="+IN"/>
 <wire x1="175.26" y1="68.58" x2="157.48" y2="68.58" width="0.1524" layer="91"/>
+<label x="160.02" y="68.58" size="1.778" layer="95"/>
+</segment>
+<segment>
+<pinref part="U$3" gate="G$1" pin="PB1(MISO)"/>
+<wire x1="119.38" y1="93.98" x2="129.54" y2="93.98" width="0.1524" layer="91"/>
+<label x="124.46" y="93.98" size="1.778" layer="95"/>
 </segment>
 </net>
@@
 </segment>
 </net>
-<net name="N$1" class="0">
+<net name="OUT1" class="0">
 <segment>
 <pinref part="U1" gate="G$1" pin="+IN"/>
 <wire x1="187.96" y1="132.08" x2="154.94" y2="132.08" width="0.1524" layer="91"/>
 <wire x1="154.94" y1="132.08" x2="154.94" y2="116.84" width="0.1524" layer="91"/>
-</segment>
-</net>
-<net name="N$4" class="0">
+<label x="157.48" y="116.84" size="1.778" layer="95"/>
+</segment>
+<segment>
+<pinref part="U$3" gate="G$1" pin="PB4(ADC2)"/>
+<wire x1="119.38" y1="86.36" x2="129.54" y2="86.36" width="0.1524" layer="91"/>
+<label x="127" y="86.36" size="1.778" layer="95"/>
+</segment>
+</net>
+<net name="N$6" class="0">
+<segment>
+<pinref part="U$3" gate="G$1" pin="PB5(NRES)"/>
+<wire x1="119.38" y1="83.82" x2="119.38" y2="73.66" width="0.1524" layer="91"/>
+<pinref part="W2R3" gate="G$1" pin="2"/>
+<wire x1="119.38" y1="73.66" x2="106.68" y2="73.66" width="0.1524" layer="91"/>
+</segment>
+</net>
+<net name="OUT2" class="0">
 <segment>
 <pinref part="U2" gate="G$1" pin="+IN"/>
 <wire x1="180.34" y1="101.6" x2="157.48" y2="101.6" width="0.1524" layer="91"/>
+<label x="160.02" y="101.6" size="1.778" layer="95"/>
+</segment>
+<segment>
+<pinref part="U$3" gate="G$1" pin="PB0(MOSI)"/>
+<wire x1="119.38" y1="96.52" x2="129.54" y2="96.52" width="0.1524" layer="91"/>
+<label x="124.46" y="96.52" size="1.778" layer="95"/>
 </segment>
 </net>
@@
 </sheet>
 </sheets>
+<errors>
+</errors>
 </schematic>
 </drawing>

Commit message: connected sch and brd
Parts:
- POTD, POTF: device LITTLEBITS140915:POT-TRIM-SMD-BOURNS-3303 -> LITTLEBITS140915:TRIMPOT_SMD_3MM
- U$6: device SparkFun_NEW:OSHW-LOGOL -> LITTLEBITS140915:OSHW-LOGOL
- W2R3: device LITTLEBITS:CAPCAP-0603 -> LITTLEBITS140915:RES-0603
Connections:
- net OUT1 renamed PB4
- net OUT2 renamed PB0
- net OUT3 renamed PB1
- removed net N$2: U$3.VCC, W2R3.1, W2U1.-IN, W2U1.OUT
- removed net N$6: U$3.PB5(NRES), W2R3.2
- new net CLN_SIG: SWITCHD.1, SWITCHF.4, W2U1.-IN, W2U1.OUT
- new net N$1: POTF.2, SWITCHF.6
- new net N$5: POTD.2, SWITCHD.3
- new net NRES: U$3.PB5(NRES), W2R3.1
- new net PB2: SWITCHD.2, U$3.PB2(SCK/ADC1)
- new net PB3: SWITCHF.5, U$3.PB3(ADC3)
- net GND: now also POTD.3, POTF.3; no longer POTD.1, POTF.1
- net VCC: now also POTD.1, POTF.1, U$3.VCC, W2R3.2; no longer POTD.3, POTF.3
Other:
- moved on the sheet: POTD, POTF, SWITCHD, SWITCHF
